File: sweepv2_custom.kicad_pcb (KiCad board)
At the start: 2 copper layers, 217.3 x 86.9 mm, 50 parts, among them J1 AudioJack4dpb, J2 AudioJack4dpb, SW10 SW_Push, SW11 SW_Push, SW11_r1 SW_Push, SW12 SW_Push, SW12_r1 SW_Push, SW13_r1 SW_Push, SW14 SW_Push, SW15 SW_Push, SW15_r1 SW_Push, SW16 SW_Push, SW16_r1 SW_Push, SW17 SW_Push, SW17_r1 SW_Push, SW18 SW_Push, SW18_r1 SW_Push, SW2 SW_Push, SW20 SW_Push, SW20_r1 SW_Push, SW21 SW_Push, SW21_r1 SW_Push, SW2_r1 SW_Push, SW3 SW_Push, SW3_r1 SW_Push, SW4 SW_Push, SW4_r1 SW_Push, SW5 SW_Push, SW5_r1 SW_Push, SW6 SW_Push, SW6_r1 SW_Push, SW7_r1 SW_Push, SW8 SW_Push, SW8_r1 SW_Push, SW9 SW_Push, SW9_r1 SW_Push, U1 ProMicro-kbd, U2 ProMicro-kbd

Commit message: Remove battery pads and overlapping silkscreen
Parts:
- moved REF** 2.18 mm to (60.4, 74.5)
- moved REF** 1.67 mm to (188.3, 75.5)

Commit message: Remove battery pads
Parts:
- removed Bat+1, Bat+r1, BatGND1, BatGND4: MountingHole_Pad, kbd:1pin_conn
- removed SW_POWER1, SW_POWERR1: SW_SPDT, Kailh:SPDT_C128955
