File: sweepv2_custom.kicad_pcb (KiCad board)
At the start: 2 copper layers, 217.3 x 86.9 mm, 44 parts, among them J1 AudioJack4dpb, J2 AudioJack4dpb, SW10 SW_Push, SW11 SW_Push, SW11_r1 SW_Push, SW12 SW_Push, SW12_r1 SW_Push, SW13_r1 SW_Push, SW14 SW_Push, SW15 SW_Push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

Commit message: Align left and right switch silkscreen image
Parts:
- moved REF** 2.59 mm to (58.0, 75.3)
- moved REF** 1.94 mm to (186.4, 75.0)
