File: sweepv2_custom.kicad_pcb (KiCad board)
At the start: 2 copper layers, 217.3 x 86.9 mm, 48 parts, among them J1 AudioJack4dpb, J2 AudioJack4dpb, SW10 SW_Push, SW11 SW_Push, SW11_r1 SW_Push, SW12 SW_Push, SW12_r1 SW_Push, SW13_r1 SW_Push, SW14 SW_Push, SW15 SW_Push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

Commit message: Remove incorrect Sweepv2 silk bottom, add custom architeuthis.dux
Parts:
- added ?: , , F.Cu at (111.7, 49.5)
