File: archive/sweepv2_custom.kicad_pcb (KiCad board)
At the start: 2 copper layers, 217.3 x 86.9 mm, 44 parts, among them J1 AudioJack4dpb, J2 AudioJack4dpb, SW10 SW_Push, SW11 SW_Push, SW11_r1 SW_Push, SW12 SW_Push, SW12_r1 SW_Push, SW13_r1 SW_Push, SW14 SW_Push, SW15 SW_Push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

Commit message: Remove unused power switch traces
Routing:
- net raw: track 0.00 -> 28.6 mm
- net gnd: track 26.1 -> 47.1 mm
- net BT+_r: track 0.00 -> 9.45 mm, vias 0 -> 1
- net BT+: track 0.00 -> 9.35 mm
