File: hypergolic V1.2 bm/hypergolic_right.kicad_pcb (KiCad board)
At the start: 2 copper layers, 119.9 x 87.7 mm, 23 parts, among them SW10 SW_Push, SW11 SW_Push, SW12 SW_Push, SW14 SW_Push, SW15 SW_Push, SW16 SW_Push, SW17 SW_Push, SW18 SW_Push, SW2 SW_Push, SW20 SW_Push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

Commit message: Add images for hypergolic 1.2bm
Parts:
-  : renamed from **
