File: hypergolic V1.2 bm/hypergolic_left.kicad_pcb (KiCad board)
At the start: 2 copper layers, 119.9 x 87.7 mm, 23 parts, among them SW10 SW_Push, SW11 SW_Push, SW12 SW_Push, SW14 SW_Push, SW15 SW_Push, SW16 SW_Push, SW17 SW_Push, SW18 SW_Push, SW2 SW_Push, SW20 SW_Push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

Commit message: Corrected traces and removed extra switch drill holes
Parts:
- added ?: , , F.Cu at (45.2, 81.0)
- added ?: , , F.Cu at (41.4, 55.6)
Changed lines of the file:
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@@
     (tracks 320)
     (zones 0)
-    (modules 23)
+    (modules 25)
     (nets 25)
   )
@@
     (add_net vcc)
   )
+  (module "" (layer F.Cu)
+    (at 45.18 81.01)
+    (fp_text reference "" (at 41.37 55.63) (layer F.SilkS)
+      (effects (font (size 1.27 1.27) (thickness 0.15)))
+    )
+    (fp_text value "" (at 41.37 55.63) (layer F.SilkS)
+      (effects (font (size 1.27 1.27) (thickness 0.15)))
+    )
+    (fp_text user BT+ (at 0.032 -1.62 180) (layer B.SilkS)
+      (effects (font (size 0.75 0.5) (thickness 0.125)) (justify mirror))
+    )
+  )
+  (module "" (layer F.Cu)
+    (at 41.37 55.63)
+    (fp_text reference "" (at 59.26 75.064) (layer F.SilkS)
+      (effects (font (size 1.27 1.27) (thickness 0.15)))
+    )
+    (fp_text value "" (at 59.26 75.064) (layer F.SilkS)
+      (effects (font (size 1.27 1.27) (thickness 0.15)))
+    )
+    (fp_text user BT+ (at 0.032 1.647 180) (layer B.SilkS)
+      (effects (font (size 0.75 0.5) (thickness 0.125)) (justify mirror))
+    )
+  )
   (module Kailh:SW_PG1350_rev_DPB (layer B.Cu)
