File: hypergolic_half/hypergolic_flip.kicad_pcb (KiCad board)
At the start: 2 copper layers, 118.8 x 87.1 mm, 24 parts, among them SW10 SW_Push, SW11 SW_Push, SW12 SW_Push, SW14 SW_Push, SW15 SW_Push, SW16 SW_Push, SW17 SW_Push, SW18 SW_Push, SW2 SW_Push, SW20 SW_Push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

Commit message: Add silkscreens
Parts:
- added REF**: silk_pg1232_bottom, silkscreens:pg1232_bottom, F.Cu at (95.3, 91.8)
- added REF**: silk_pg2132_top, silkscreens:pg1232_top, B.Cu at (95.3, 91.8)
