File: macro3/macro3.kicad_pcb (KiCad board)
At the start: 2 copper layers, 95.6 x 40.7 mm, 9 parts, among them SW1 SW_PUSH, SW2 SW_PUSH, SW5 SW_PUSH, SW6 SW_PUSH, SW7 Rotary_Encoder_Switch, SW7 SW_PUSH, SW8 SW_PUSH, U1 ProMicro_r

Commit message: Remove encoder silk
Parts:
-  : renamed from SW7 (x2)
