File: hypergarlic/hypergarlic_update.kicad_pcb (KiCad board)
At the start: 2 copper layers, 238.8 x 87.7 mm, 40 parts, among them J1 AudioJack4dpb, J2 AudioJack4dpb, SW10 SW_Push, SW11 SW_Push, SW11_r1 SW_Push, SW12 SW_Push, SW12_r1 SW_Push, SW13_r1 SW_Push, SW14 SW_Push, SW15 SW_Push, SW15_r1 SW_Push, SW16 SW_Push, SW16_r1 SW_Push, SW17 SW_Push, SW17_r1 SW_Push, SW18 SW_Push, SW18_r1 SW_Push, SW2 SW_Push, SW20 SW_Push, SW20_r1 SW_Push, SW21 SW_Push, SW21_r1 SW_Push, SW2_r1 SW_Push, SW3 SW_Push, SW3_r1 SW_Push, SW4 SW_Push, SW4_r1 SW_Push, SW5 SW_Push, SW5_r1 SW_Push, SW6 SW_Push, SW6_r1 SW_Push, SW7_r1 SW_Push, SW8 SW_Push, SW8_r1 SW_Push, SW9 SW_Push, SW9_r1 SW_Push, U1 ProMicro-kbd, U2 ProMicro-kbd

Commit message: Remove clove, add silkscreen image
Parts:
- added REF**: silk_pg1232_footprint, silkscreens:pg1232_footprint, B.Cu at (199.5, 95.0)
- added REF**: silk_pg1232_bottom, silkscreens:pg1232_bottom, B.Cu at (81.4, 95.0)
- added REF**: silk_pg2132_top, silkscreens:pg1232_top, B.Cu at (62.3, 94.8)
