File: hypergarlic/hypergarlic_update.kicad_pcb (KiCad board)
At the start: 2 copper layers, 238.8 x 87.7 mm, 43 parts, among them J1 AudioJack4dpb, J2 AudioJack4dpb, SW10 SW_Push, SW11 SW_Push, SW11_r1 SW_Push, SW12 SW_Push, SW12_r1 SW_Push, SW13_r1 SW_Push, SW14 SW_Push, SW15 SW_Push, SW15_r1 SW_Push, SW16 SW_Push, SW16_r1 SW_Push, SW17 SW_Push, SW17_r1 SW_Push, SW18 SW_Push, SW18_r1 SW_Push, SW2 SW_Push, SW20 SW_Push, SW20_r1 SW_Push, SW21 SW_Push, SW21_r1 SW_Push, SW2_r1 SW_Push, SW3 SW_Push, SW3_r1 SW_Push, SW4 SW_Push, SW4_r1 SW_Push, SW5 SW_Push, SW5_r1 SW_Push, SW6 SW_Push, SW6_r1 SW_Push, SW7_r1 SW_Push, SW8 SW_Push, SW8_r1 SW_Push, SW9 SW_Push, SW9_r1 SW_Push, U1 ProMicro-kbd, U2 ProMicro-kbd

Commit message: Add Paroxysm and update hypergarlic gerber
Routing:
- net gnd: track 8.25 -> 4.11 mm
Changed lines of the file:
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@@
     (thickness 1.6)
     (drawings 52)
-    (tracks 687)
+    (tracks 685)
     (zones 0)
     (modules 43)
@@
   (segment (start 152.1914 51.324) (end 152.1914 53.864) (width 0.25) (layer B.Cu) (net 1))
   (segment (start 133.428401 50.212999) (end 132.3174 51.324) (width 0.25) (layer B.Cu) (net 1))
-  (segment (start 135.542401 50.212999) (end 133.428401 50.212999) (width 0.25) (layer B.Cu) (net 1))
-  (segment (start 136.9714 48.784) (end 135.542401 50.212999) (width 0.25) (layer B.Cu) (net 1))
   (segment (start 140.868 78.218) (end 141.492 78.218) (width 0.25) (layer B.Cu) (net 2))
   (segment (start 126.608 84.582) (end 125.03 84.582) (width 0.25) (layer B.Cu) (net 2))
