File: Architeuthis dux/architeuthis_dux_filled.kicad_pcb (KiCad board)
At the start: 2 copper layers, 129.9 x 95.6 mm, 19 parts

Commit message: Remove half-swept
Routing:
- net GND: track 944.7 -> 23.6 mm
- net P6: track 140.4 -> 142.0 mm
Other:
- outline, holes or cut-outs redrawn
- net class Default removed
