File: Sweep High/sweep-high-combo.kicad_pcb (KiCad board)
At the start: 2 copper layers, 229.5 x 95.2 mm, 42 parts, among them J1 AudioJack4dpb, J2 AudioJack4dpb, SW10 SW_Push, SW11 SW_Push, SW11_r1 SW_Push, SW12 SW_Push, SW12_r1 SW_Push, SW13_r1 SW_Push, SW14 SW_Push, SW15 SW_Push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

Commit message: Update and corrected traces
Routing:
- net gnd: track 5.95 -> 0.75 mm
- net Switch6_r: track 158.0 -> 156.6 mm
- net Switch4_r: track 67.3 -> 67.9 mm
- net Switch10: track 44.4 -> 43.8 mm
- net Switch18_r: vias 1 -> 0
Other:
- net class Default removed
