File: hypergolic V1.4 high/hypergolic_high.kicad_pcb (KiCad board)
At the start: 2 copper layers, 125.5 x 95.5 mm, 21 parts, among them SW10 SW_Push, SW11 SW_Push, SW12 SW_Push, SW14 SW_Push, SW15 SW_Push, SW16 SW_Push, SW17 SW_Push, SW18 SW_Push, SW2 SW_Push, SW20 SW_Push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

Commit message: Add stemcell
Parts:
- removed REF**: Tenting Puck, kbd:Tenting_Puck2
- removed RSW1: SW_Push, kbd:ResetSW
Routing:
- net reset: track 71.8 -> 0.00 mm
