File: Sweep/sweepv21_minimal.kicad_pcb (KiCad board)
At the start: 2 copper layers, 217.4 x 86.9 mm, 40 parts, among them J1 AudioJack4dpb, J2 AudioJack4dpb, SW10 SW_Push, SW11 SW_Push, SW11_r1 SW_Push, SW12 SW_Push, SW12_r1 SW_Push, SW13_r1 SW_Push, SW14 SW_Push, SW15 SW_Push, SW15_r1 SW_Push, SW16 SW_Push, SW16_r1 SW_Push, SW17 SW_Push, SW17_r1 SW_Push, SW18 SW_Push, SW18_r1 SW_Push, SW2 SW_Push, SW20 SW_Push, SW20_r1 SW_Push, SW21 SW_Push, SW21_r1 SW_Push, SW2_r1 SW_Push, SW3 SW_Push, SW3_r1 SW_Push, SW4 SW_Push, SW4_r1 SW_Push, SW5 SW_Push, SW5_r1 SW_Push, SW6 SW_Push, SW6_r1 SW_Push, SW7_r1 SW_Push, SW8 SW_Push, SW8_r1 SW_Push, SW9 SW_Push, SW9_r1 SW_Push, U1 ProMicro-kbd, U2 ProMicro-kbd

Commit message: Add modified left and right only paroxysm
Parts:
- added REF**: LOGO, silkscreens:safe_rust, B.Cu at (80.6, 47.8)
- added REF**: LOGO, silkscreens:unsafe_rust, B.Cu at (180.9, 54.1)
Other:
- net class Default removed

Commit message: Add splinter pcb
Routing:
- net gnd: track 86.3 -> 45.6 mm
- net reset_r: track 38.0 -> 0.00 mm, vias 1 -> 0
- net reset: track 27.3 -> 0.00 mm, vias 1 -> 0
